Commit message: edited the joint order to match the ros2-controls hardware interface

File: src/diffbot_description/urdf/diffbot_ros2_control.xacro (robot description, xacro)
@@ -5,5 +5,5 @@
       <plugin>gz_ros2_control/GazeboSimSystem</plugin>
     </hardware>
-    <joint name="left_wheel_joint">
+    <joint name="right_wheel_joint">
       <command_interface name="velocity">
         <param name="min">-10</param>
@@ -13,5 +13,5 @@
       <state_interface name="position"/>
     </joint>
-    <joint name="right_wheel_joint">
+    <joint name="left_wheel_joint">
       <command_interface name="velocity">
         <param name="min">-10</param>
